Commit message: Add visualisation for right handed glove.

File: urdf/righthand_NED.xacro (robot description, xacro)
@@ -1,4 +1,4 @@
 <?xml version="1.0" ?>
-<robot name = "righthand" xmlns:xacro="http://ros.org/wiki/xacro">
+<robot name = "lefthand" xmlns:xacro="http://ros.org/wiki/xacro">
     <!-- Include Materials -->
     <material name="Black">
@@ -16,4 +16,5 @@
     <xacro:property name="M_PI" value="3.14159"/>
     <xacro:property name="rpy" value="1.57 0 1.57"/>
+    <!-- BODY -->
     <!-- Carpals Box -->
     <xacro:property name="c_l" value="0.0437" />
@@ -21,5 +22,4 @@
     <xacro:property name="c_h" value="0.02" />
     <!-- Metacarpals Box-->
-    <xacro:property name="x_origin" value="0.5" />
     <xacro:property name="metc_l" value="0.16" />
     <xacro:property name="metc_b" value="0.025" />
@@ -43,5 +43,5 @@
         <transmission name="tran1">
             <type>transmission_interface/SimpleTransmission</type>
-            <joint name="${joint_name}">
+            <joint name="${prefix}_${joint_name}">
     	      <hardwareInterface>hardware_interface/PositionJointInterface</hardwareInterface>
             </joint>
@@ -52,328 +52,351 @@
         </transmission>
     </xacro:macro>
-    <!-- /////////////////////////////////////////////////////////////////////////////// -->
     <!-- JOINTS AND LINKS -->
-<!--    -->
-    <link name="metacarpal">
-        <visual>
-            <origin xyz="${x_origin+0.05185} 0 0" rpy="${rpy}"/>
-            <geometry>
-                <box size="${metc_l} ${metc_b} ${metc_h}"/>
-            </geometry>
-            <material name="White"/>
-        </visual>
-<!--        <xacro:inertial_matrix mass="1"/>-->
-    </link>
-    <gazebo reference="metacarpal">
-        <material>Gazebo/Black</material>
-    </gazebo>
+    <!-- XACRO:MACRO HAND -->
+    <xacro:macro name="hand" params="prefix reflect metacarpal_origin_x">
+<!--        <joint name="body_to_${prefix}_metacarpal" type="floating">-->
+<!--            <origin xyz="${reflect*(metacarpal_origin_x-0.06)} 0.08 0.0125" rpy="-1.57 0 0"/>-->
+<!--            <parent link="body"/>-->
+<!--            <child link="${prefix}_metacarpal"/>-->
+<!--            <axis xyz="0 0 1"/>-->
+<!--            &lt;!&ndash;        <limit effort="300" velocity="1" lower="-1.57" upper="0" />&ndash;&gt;-->
+<!--            <dynamics damping="50" friction="1"/>-->
+<!--        </joint>-->
+    <!--    -->
+        <link name="${prefix}_metacarpal">
+            <visual>
+                <origin xyz="${reflect*(0.05185)} 0 0" rpy="${rpy}"/>
+                <geometry>
+                    <box size="${metc_l} ${metc_b} ${metc_h}"/>
+                </geometry>
+                <material name="White"/>
+            </visual>
+    <!--        <xacro:inertial_matrix mass="1"/>-->
+        </link>
+        <gazebo reference="${prefix}_metacarpal">
+            <material>Gazebo/Black</material>
+        </gazebo>
+        <!-- ///////////////////////////////////////////////////////////////////////////////////////////////////////////////////// -->
+         <!-- THUMB FINGER PROXIMAL-->
+        <joint name="${prefix}_metacarpal_thumb_splay_2" type="continuous">
+            <origin xyz="${reflect*(0.06)} 0.08 0.0125" rpy="-1.57 0 0"/>
+            <parent link="${prefix}_metacarpal"/>
+            <child link="${prefix}_thumb_p_splay2"/>
+            <axis xyz="0 0 -1"/>
+            <!--        <limit effort="300" velocity="1" lower="-1.57" upper="0" />-->
+            <dynamics damping="50" friction="1"/>
+        </joint>
+        <link name="${prefix}_thumb_p_splay2"></link>  <!-- SPLAY 2 LINK -->
+        <!-- THUMB FINGER PROXIMAL-->
+        <joint name="${prefix}_thumb_meta_prox" type="continuous">
+            <origin xyz="${reflect*0} 0 0" rpy="0 0 0"/>
+            <parent link="${prefix}_thumb_p_splay2"/>
+            <child link="${prefix}_thumb_p"/>
+            <axis xyz="0 1 0"/>
+            <!--        <limit effort="300" velocity="1" lower="-1.57" upper="0" />-->
+            <dynamics damping="50" friction="1"/>
+        </joint>
+        <link name="${prefix}_thumb_p">
+            <visual>
+                <origin xyz="${reflect*(0.018)} 0 0" rpy="1.57 0 1.57"/>
+                <geometry>
+                    <cylinder radius="${proxrad}" length="${proxlen}"/>
+                </geometry>
+                <material name="White"/>
+            </visual>
+            <xacro:inertial_matrix mass="1"/>
+        </link>
+        <!-- THUMB FINGER INTERMEDIATE-->
+        <joint name="${prefix}_thumb_prox_inter" type="continuous">
+            <origin xyz="${proxlen} 0 0" rpy="0 0 0"/>
+            <parent link="${prefix}_thumb_p"/>
+            <child link="${prefix}_thumb_i"/>
+            <axis xyz="0 1 0"/>
+            <!--        <limit effort="300" velocity="1" lower="-1.57" upper="0" />-->
+            <dynamics damping="50" friction="1"/>
+        </joint>
+        <link name="${prefix}_thumb_i">
+            <visual>
+                <origin xyz="${reflect*(0.018)} 0 0" rpy="0 1.57 0"/>
+                <geometry>
+                    <cylinder radius="${interrad}" length="${interlen}"/>
+                </geometry>
+                <material name="White"/>
+            </visual>
+            <xacro:inertial_matrix mass="1"/>
+        </link>
+    <!-- THUMB END -->
+        <!-- INDEX FINGER PROXIMAL-->
+        <joint name="${prefix}_metacarpal_index" type="continuous">
+            <origin xyz="${reflect*(0.0937)} 0 0" rpy="0 0 0"/>
+            <parent link="${prefix}_metacarpal"/>
+            <child link="${prefix}_index_p"/>
+            <axis xyz="0 -1 0"/>
+            <!--        <limit effort="300" velocity="1" lower="-1.57" upper="0" />-->
+            <dynamics damping="50" friction="1"/>
+        </joint>
+        <link name="${prefix}_index_p">
+            <visual>
+                <origin xyz="${reflect*(0.018)} 0.055 0" rpy="${rpy}"/>
+                <geometry>
+                    <cylinder radius="${proxrad}" length="${proxlen}"/>
+                </geometry>
+                <material name="White"/>
+            </visual>
+            <xacro:inertial_matrix mass="1"/>
+        </link>
+        <!-- INDEX FINGER INTERMEDIATE-->
+        <joint name="${prefix}_index_prox_inter" type="continuous">
+            <origin xyz="${proxlen} 0 0" rpy="0 0 0"/>
+            <parent link="${prefix}_index_p"/>
+            <child link="${prefix}_index_i"/>
+            <axis xyz="0 -1 0"/>
+            <!--        <limit effort="300" velocity="1" lower="-1.57" upper="0" />-->
+            <dynamics damping="50" friction="1"/>
+        </joint>
+        <link name="${prefix}_index_i">
+            <visual>
+                <origin xyz="${reflect*(0.016)} 0.055 0" rpy="${rpy}"/>
+                <geometry>
+                    <cylinder radius="${interrad}" length="${interlen}"/>
+                </geometry>
+                <material name="White"/>
+            </visual>
+            <xacro:inertial_matrix mass="1"/>
+        </link>
+        <!-- INDEX FINGER DISTAL-->
+        <joint name="${prefix}_index_inter_dist" type="continuous">
+            <origin xyz="${interlen} 0 0" rpy="0 0 0"/>
+            <parent link="${prefix}_index_i"/>
+            <child link="${prefix}_index_d"/>
+            <axis xyz="0 -1 0"/>
+            <!--        <limit effort="300" velocity="1" lower="-1.57" upper="0" />-->
+            <dynamics damping="50" friction="1"/>
+        </joint>
+        <link name="${prefix}_index_d">
+            <visual>
+                <origin xyz="${reflect*(0.020)} 0.055 0" rpy="${rpy}"/>
+                <geometry>
+                    <cylinder radius="${distrad}" length="${distlen}"/>
+                </geometry>
+                <material name="White"/>
+            </visual>
+            <xacro:inertial_matrix mass="1"/>
+        </link>
+        <!-- ///////////////////////////////////////////////////////////////////////////////////////////////////////////////////// -->
+        <!-- MIDDLE FINGER PROXIMAL-->
+        <joint name="${prefix}_metacarpal_middle" type="continuous">
+            <origin xyz="${reflect*(0.0937)} 0 0" rpy="0 0 0"/>
+            <parent link="${prefix}_metacarpal"/>
+            <child link="${prefix}_middle_p"/>
+            <axis xyz="0 -1 0"/>
+            <!--        <limit effort="300" velocity="1" lower="-1.57" upper="0" />-->
+            <dynamics damping="50" friction="1"/>
+        </joint>
+        <link name="${prefix}_middle_p">
+            <visual>
+                <origin xyz="${reflect*(0.018)} 0.0225 0" rpy="${rpy}"/>
+                <geometry>
+                    <cylinder radius="${proxrad}" length="${proxlen}"/>
+                </geometry>
+                <material name="White"/>
+            </visual>
+            <xacro:inertial_matrix mass="1"/>
+        </link>
+        <!-- MIDDLE FINGER INTERMEDIATE-->
+        <joint name="${prefix}_middle_prox_inter" type="continuous">
+            <origin xyz="${proxlen} 0 0" rpy="0 0 0"/>
+            <parent link="${prefix}_middle_p"/>
+            <child link="${prefix}_middle_i"/>
+            <axis xyz="0 -1 0"/>
+            <!--        <limit effort="300" velocity="1" lower="-1.57" upper="0" />-->
+            <dynamics damping="50" friction="1"/>
+        </joint>
+        <link name="${prefix}_middle_i">
+            <visual>
+                <origin xyz="${reflect*(0.016)} 0.0225 0" rpy="${rpy}"/>
+                <geometry>
+                    <cylinder radius="${interrad}" length="${interlen}"/>
+                </geometry>
+                <material name="White"/>
+            </visual>
+            <xacro:inertial_matrix mass="1"/>
+        </link>
+        <!-- MIDDLE FINGER DISTAL-->
+        <joint name="${prefix}_middle_inter_dist" type="continuous">
+            <origin xyz="${interlen} 0 0" rpy="0 0 0"/>
+            <parent link="${prefix}_middle_i"/>
+            <child link="${prefix}_middle_d"/>
+            <axis xyz="0 -1 0"/>
+            <!--        <limit effort="300" velocity="1" lower="-1.57" upper="0" />-->
+            <dynamics damping="50" friction="1"/>
+        </joint>
+        <link name="${prefix}_middle_d">
+            <visual>
+                <origin xyz="${reflect*(0.025)} 0.0225 0" rpy="${rpy}"/>
+                <geometry>
+                    <cylinder radius="${distrad}" length="${distlen - 0.01}"/>
+                </geometry>
+                <material name="White"/>
+            </visual>
+            <xacro:inertial_matrix mass="1"/>
+        </link>
     <!-- ///////////////////////////////////////////////////////////////////////////////////////////////////////////////////// -->
-     <!-- THUMB FINGER PROXIMAL-->
-    <joint name="metacarpal_thumb_splay_2" type="continuous">
-        <origin xyz="${x_origin+0.06} 0.08 0.0125" rpy="-1.57 0 0"/>
-        <parent link="metacarpal"/>
-        <child link="thumb_p_splay2"/>
-        <axis xyz="0 0 1"/>
-        <!--        <limit effort="300" velocity="1" lower="-1.57" upper="0" />-->
-        <dynamics damping="50" friction="1"/>
-    </joint>
-    <link name="thumb_p_splay2"></link>  <!-- SPLAY 2 LINK -->
-    <!-- THUMB FINGER PROXIMAL-->
-    <joint name="thumb_meta_prox" type="continuous">
-        <origin xyz="${x_origin} 0 0" rpy="0 0 0"/>
-        <parent link="thumb_p_splay2"/>
-        <child link="thumb_p"/>
-        <axis xyz="0 1 0"/>
-        <!--        <limit effort="300" velocity="1" lower="-1.57" upper="0" />-->
-        <dynamics damping="50" friction="1"/>
-    </joint>
-    <link name="thumb_p">
-        <visual>
-            <origin xyz="${x_origin+0.018} 0 0" rpy="1.57 0 1.57"/>
-            <geometry>
-                <cylinder radius="${proxrad}" length="${proxlen}"/>
-            </geometry>
-            <material name="White"/>
-        </visual>
-        <xacro:inertial_matrix mass="1"/>
-    </link>
-    <!-- THUMB FINGER INTERMEDIATE-->
-    <joint name="thumb_prox_inter" type="continuous">
-        <origin xyz="${x_origin+proxlen} 0 0" rpy="0 0 0"/>
-        <parent link="thumb_p"/>
-        <child link="thumb_i"/>
-        <axis xyz="0 1 0"/>
-        <!--        <limit effort="300" velocity="1" lower="-1.57" upper="0" />-->
-        <dynamics damping="50" friction="1"/>
-    </joint>
-    <link name="thumb_i">
-        <visual>
-            <origin xyz="${x_origin+0.018} 0 0" rpy="0 1.57 0"/>
-            <geometry>
-                <cylinder radius="${interrad}" length="${interlen}"/>
-            </geometry>
-            <material name="White"/>
-        </visual>
-        <xacro:inertial_matrix mass="1"/>
-    </link>
-<!-- THUMB END -->
-    <!-- INDEX FINGER PROXIMAL-->
-    <joint name="metacarpal_index" type="continuous">
-        <origin xyz="${x_origin+0.0937} 0 0" rpy="0 0 0"/>
-        <parent link="metacarpal"/>
-        <child link="index_p"/>
-        <axis xyz="0 1 0"/>
-        <!--        <limit effort="300" velocity="1" lower="-1.57" upper="0" />-->
-        <dynamics damping="50" friction="1"/>
-    </joint>
-    <link name="index_p">
-        <visual>
-            <origin xyz="${x_origin+0.018} 0.055 0" rpy="${rpy}"/>
-            <geometry>
-                <cylinder radius="${proxrad}" length="${proxlen}"/>
-            </geometry>
-            <material name="White"/>
-        </visual>
-        <xacro:inertial_matrix mass="1"/>
-    </link>
-    <!-- INDEX FINGER INTERMEDIATE-->
-    <joint name="index_prox_inter" type="continuous">
-        <origin xyz="${x_origin+proxlen} 0 0" rpy="0 0 0"/>
-        <parent link="index_p"/>
-        <child link="index_i"/>
-        <axis xyz="0 1 0"/>
-        <!--        <limit effort="300" velocity="1" lower="-1.57" upper="0" />-->
-        <dynamics damping="50" friction="1"/>
-    </joint>
-    <link name="index_i">
-        <visual>
-            <origin xyz="${x_origin+0.016} 0.055 0" rpy="${rpy}"/>
-            <geometry>
-                <cylinder radius="${interrad}" length="${interlen}"/>
-            </geometry>
-            <material name="White"/>
-        </visual>
-        <xacro:inertial_matrix mass="1"/>
-    </link>
-    <!-- INDEX FINGER DISTAL-->
-    <joint name="index_inter_dist" type="continuous">
-        <origin xyz="${x_origin+interlen} 0 0" rpy="0 0 0"/>
-        <parent link="index_i"/>
-        <child link="index_d"/>
-        <axis xyz="0 1 0"/>
-        <!--        <limit effort="300" velocity="1" lower="-1.57" upper="0" />-->
-        <dynamics damping="50" friction="1"/>
-    </joint>
-    <link name="index_d">
-        <visual>
-            <origin xyz="${x_origin+0.020} 0.055 0" rpy="${rpy}"/>
-            <geometry>
-                <cylinder radius="${distrad}" length="${distlen}"/>
-            </geometry>
-            <material name="White"/>
-        </visual>
-        <xacro:inertial_matrix mass="1"/>
-    </link>
+        <!-- ///////////////////////////////////////////////////////////////////////////////////////////////////////////////////// -->
+        <!-- RING FINGER PROXIMAL-->
+        <joint name="${prefix}_metacarpal_ring" type="continuous">
+            <origin xyz="${reflect*(0.0937)} 0 0" rpy="0 0 0"/>
+            <parent link="${prefix}_metacarpal"/>
+            <child link="${prefix}_ring_p"/>
+            <axis xyz="0 -1 0"/>
+            <!--        <limit effort="300" velocity="1" lower="-1.57" upper="0" />-->
+            <dynamics damping="50" friction="1"/>
+        </joint>
+        <link name="${prefix}_ring_p">
+            <visual>
+                <origin xyz="${reflect*(0.018)} -0.0225 0" rpy="${rpy}"/>
+                <geometry>
+                    <cylinder radius="${proxrad}" length="${proxlen}"/>
+                </geometry>
+                <material name="White"/>
+            </visual>
+            <xacro:inertial_matrix mass="1"/>
+        </link>
+        <!-- RING FINGER INTERMEDIATE-->
+        <joint name="${prefix}_ring_prox_inter" type="continuous">
+            <origin xyz="${proxlen} 0 0" rpy="0 0 0"/>
+            <parent link="${prefix}_ring_p"/>
+            <child link="${prefix}_ring_i"/>
+            <axis xyz="0 -1 0"/>
+            <!--        <limit effort="300" velocity="1" lower="-1.57" upper="0" />-->
+            <dynamics damping="50" friction="1"/>
+        </joint>
+        <link name="${prefix}_ring_i">
+            <visual>
+                <origin xyz="${reflect*(0.016)} -0.0225 0" rpy="${rpy}"/>
+                <geometry>
+                    <cylinder radius="${interrad}" length="${interlen}"/>
+                </geometry>
+                <material name="White"/>
+            </visual>
+            <xacro:inertial_matrix mass="1"/>
+        </link>
+        <!-- RING FINGER DISTAL-->
+        <joint name="${prefix}_ring_inter_dist" type="continuous">
+            <origin xyz="${interlen} 0 0" rpy="0 0 0"/>
+            <parent link="${prefix}_ring_i"/>
+            <child link="${prefix}_ring_d"/>
+            <axis xyz="0 -1 0"/>
+            <!--        <limit effort="300" velocity="1" lower="-1.57" upper="0" />-->
+            <dynamics damping="50" friction="1"/>
+        </joint>
+        <link name="${prefix}_ring_d">
+            <visual>
+                <origin xyz="${reflect*(0.020)} -0.0225 0" rpy="${rpy}"/>
+                <geometry>
+                    <cylinder radius="${distrad}" length="${distlen}"/>
+                </geometry>
+                <material name="White"/>
+            </visual>
+            <xacro:inertial_matrix mass="1"/>
+        </link>
+        <!-- ///////////////////////////////////////////////////////////////////////////////////////////////////////////////////// -->
+        <!-- PINKY FINGER PROXIMAL-->
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